Commit message: 新增碰撞体，防止yaw碰撞

File: assets/ultra_GameYaw/urdf/ultra0523Yaw.urdf (robot description, URDF)
Before this commit: robot urdf0523P2, 14 links, 13 joints
Links:
- link hip_roll_l_link: geometry collision cylinder length=0.1475 radius=0.065; visual mesh filename=../meshes/hip_roll_l_link.STL
- link hip_roll_r_link: geometry collision cylinder length=0.1475 radius=0.065; visual mesh filename=../meshes/hip_roll_r_link.STL
